File: board/hw_design/MARK-II board.brd (EAGLE design)
At the start: 130 x 80 mm, 169 parts, among them IC1 MAX3243CPWR, IC10 IFX1963TBV, IC11 IFX1963TBV, IC12 ATMEGA48PB-AU, IC13 LD1117S33, IC2 FT230XS, IC3 ENC28J60SS, IC4 PCM5100, IC5 AS4C32M8SA, IC6 MCP7940NSN, IC7 FM24CL16BG, IC8 AT25DN256SS, IC9 10M25SAE144, Q1 25MHz, Q2 32.768kHz, Q3 CMI-1275C-050, Q4 25MHz, Q5 18,432MHz, Q6 22.5792MHz, T1 BC337-16 A1, X1 MINI-USBUX60A-MB-5ST, X10 T821-106A1S100, X11 T821-110A1S100, X12 PJ-002BH-SMT-TR, X13 T821-106A1S100, X2 5504F1-09P-02A-03, X3 L77HDE15SD1CH4R, X4 MD-60SM, X5 RB1-125BAG1A, X6 SJ1-3535NG, X7 MICROSD-HRS_DM3D, X8 BAT-HLD-002-SMT, X9 T821-120A1S100

Commit message: Changed LDO
Parts:
- IC10, IC11: value IFX1963TBV -> MIC29302A
Changed lines of the file:
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@@
 <attribute name="VALUE" x="100.965" y="48.895" size="1.27" layer="27" rot="R90"/>
 </element>
-<element name="IC10" library="vreg" package="D2PAK-5" value="IFX1963TBV" x="8.89" y="57.15" smashed="yes">
-<attribute name="MOUSER" value="726-IFX1963TBV" x="8.89" y="57.15" size="1.778" layer="27" display="off"/>
+<element name="IC10" library="vreg" package="D2PAK-5" value="MIC29302A" x="8.89" y="57.15" smashed="yes">
+<attribute name="MOUSER" value="998-MIC29302AWU" x="8.89" y="57.15" size="1.778" layer="27" display="off"/>
 <attribute name="NAME" x="8.89" y="48.26" size="1.27" layer="25" font="vector" align="center"/>
 <attribute name="VALUE" x="16.51" y="56.515" size="1.27" layer="27" rot="R90"/>
 </element>
-<element name="IC11" library="vreg" package="D2PAK-5" value="IFX1963TBV" x="22.86" y="57.15" smashed="yes">
-<attribute name="MOUSER" value="726-IFX1963TBV" x="22.86" y="57.15" size="1.778" layer="27" display="off"/>
+<element name="IC11" library="vreg" package="D2PAK-5" value="MIC29302A" x="22.86" y="57.15" smashed="yes">
+<attribute name="MOUSER" value="998-MIC29302AWU" x="22.86" y="57.15" size="1.778" layer="27" display="off"/>
 <attribute name="NAME" x="22.86" y="48.26" size="1.27" layer="25" font="vector" align="center"/>
 <attribute name="VALUE" x="30.48" y="56.515" size="1.27" layer="27" rot="R90"/>
